File: PCB/Roto-Pad_SeeedXiaoBLE/Roto-Pad_SeeedXiaoBLE.kicad_sch (KiCad schematic)
At the start: 62 parts

Commit message: seeed PCB completed
Parts:
- removed B?: SPARKFUN_PRO_MICRO, Boards:SPARKFUN_PRO_MICRO, symbol SparkFun-Boards:SPARKFUN_PRO_MICRO
- removed D? (x25): DIODE-1N4148, Custom:D_0805_2012Metric_Pad1.15x1.40mm_HandSolder, symbol SparkFun-DiscreteSemi:DIODE-1N4148
- removed J?: I2C_STANDARD_NO_SILK, Connectors:1X04_NO_SILK, symbol SparkFun-Connectors:I2C_STANDARD_NO_SILK
- removed S?: MOMENTARY-SWITCH-SPST-2-SMD-4.6X2.8MM, Switches:TACTILE_SWITCH_SMD_4.6X2.8MM, symbol SparkFun-Switches:MOMENTARY-SWITCH-SPST-2-SMD-4.6X2.8MM
- removed SW? (x23): HECKIN_LED_SWITCH, Custom:xX_Super_Heckin_Valid_MX_CHOC_SK6812MINIE_ONESIDE_KEYSWITCH_UwU_Xx, symbol Universal_Keyswitch:HECKIN_LED_SWITCH
- removed SW? (x2): RotarySwitchLedHybrid, Custom:xX_Super_Heckin_Valid_Rotary_MX_Kailh_Hybrid_UwU_Xx, symbol Custom:RotarySwitchLedHybrid
- added BT1: Battery, Custom:804040 LiPo, symbol Device:Battery
- added I1: I2C_OLED, Custom:TINY OLED I2C, symbol Custom:I2C_OLED
- added P1, P3: Pin_R, TestPoint:TestPoint_THTPad_D2.0mm_Drill1.0mm, symbol Custom:Pin_R
- added P2, P4: Pin_S, TestPoint:TestPoint_THTPad_2.0x2.0mm_Drill1.0mm, symbol Custom:Pin_S
- added SW1, SW5: LedRotary_Neopixel_Switch_Hybrid, Custom:xX_Super_Heckin_Valid_LED_Rotory_Neopixel_Kailh_MX_Keyswitch_UwU_Xx, symbol Custom:LedRotary_Neopixel_Switch_Hybrid
- added SW10, SW11, SW12, SW13, SW14, SW15, SW16, SW17, SW18, SW19, SW2, SW20, SW21, SW22, SW23, SW24, SW25, SW3, SW4, SW6, SW7, SW8, SW9: Heckin_LED_Switch, Custom:xX_Super_Heckin_Valid_MX_CHOC_SK6812MINIE_ONESIDE_KEYSWITCH_UwU_Xx, symbol Custom:Heckin_LED_Switch
- added U1: PCA9506BS,118, eec:NXP_Semiconductors-PCA9506BS,118-Manufacturer_Recommended, symbol eec:PCA9506BS,118
- added U2: XIAOBLE, Seeeduino XIAO KICAD:Seeeduino XIAO-MOUDLE14P-2.54-21X17.8MM, symbol Seeeduino XIAO:XIAOBLE
- C1: renamed from C?; footprint Capacitor_THT:C_Axial_L5.1mm_D3.1mm_P12.50mm_Horizontal -> Capacitors:1210
- LED1, LED2, LED3, LED4, LED5, LED6, LED7, LED8: renamed from LED?; footprint Keebio-Parts:WS2812B-4020 -> Custom:Neopixel 2040
Connections:
- net +5V is gone; now on net 5V: C1.1
- net 5V: now also I1.2 (VCC), SW1.1 (Sw1), SW1.5v, SW10.1 (Sw1), SW10.5v, SW11.1 (Sw1), SW11.5v, SW12.1 (Sw1), SW12.5v, SW13.1 (Sw1), SW13.5v, SW14.1 (Sw1), SW14.5v, SW15.1 (Sw1), SW15.5v, SW16.1 (Sw1), SW16.5v, SW17.1 (Sw1), SW17.5v, SW18.1 (Sw1), SW18.5v, SW19.1 (Sw1), SW19.5v, SW2.1 (Sw1), SW2.5v, SW20.1 (Sw1), SW20.5v, SW21.1 (Sw1), SW21.5v, SW22.1 (Sw1), SW22.5v, SW23.1 (Sw1), SW23.5v, SW24.1 (Sw1), SW24.5v, SW25.1 (Sw1), SW25.5v, SW3.1 (Sw1), SW3.5v, SW4.1 (Sw1), SW4.5v, SW5.1 (Sw1), SW5.5v, SW6.1 (Sw1), SW6.5v, SW7.1 (Sw1), SW7.5v, SW8.1 (Sw1), SW8.5v, SW9.1 (Sw1), SW9.5v, U1.11 (VDD), U1.20 (A0), U1.39 (VDD), U1.49 (~{RESET}), U2.14 (5V)
- net Earth: now also I1.1 (GND), SW1.C, SW1.GND, SW10.GND, SW11.GND, SW12.GND, SW13.GND, SW14.GND, SW15.GND, SW16.GND, SW17.GND, SW18.GND, SW19.GND, SW2.GND, SW20.GND, SW21.GND, SW22.GND, SW23.GND, SW24.GND, SW25.GND, SW3.GND, SW4.GND, SW5.C, SW5.GND, SW6.GND, SW7.GND, SW8.GND, SW9.GND, U1.16 (VSS), U1.21 (A1), U1.22 (A2), U1.27 (VSS), U1.3 (IO0_6), U1.32 (VSS), U1.4 (VSS), U1.44 (VSS), U1.45 (IO4_5), U1.46 (IO4_6), U1.47 (IO4_7), U1.5 (IO0_7), U1.55 (VSS), U1.57 (EP), U2.13 (GND), U2.20 (GND)
- net LED CONTROL: now also SW1.DIN, U2.4 (PA11_A3_D3)
- net Rot 2 A: now also SW5.A, U1.36 (IO3_6)
- net Rot1 A: now also SW1.A, U1.6 (IO1_0)
- net Rot1B: now also SW1.B, U1.7 (IO1_1)
- net Rot2B: now also SW5.B, U1.37 (IO3_7)
- net SCL: now also I1.3 (SCL), P4.1, U1.50 (SDA), U2.6 (PA9_A5_D5_SCL)
- net SDA: now also I1.4 (SDA), P3.1, U1.51 (SCL), U2.5 (PA8_A4_D4_SDA)
- net Ledthru renamed LEDROW5
- net LEDROW5: now also SW25.DOUT
- net Ledthru2: no longer names the net of LED4.4 (DOUT), LED5.2 (DIN)
- new net: SW19.DOUT, SW20.DIN
- new net: BT1.2 (-), U2.21 (Batt-)
- new net: BT1.1 (+), U2.22 (Batt_+)
- new net: SW21.DOUT, SW22.DIN
- new net: SW13.DOUT, SW14.DIN
- new net: SW14.DOUT, SW15.DIN
- new net: SW16.DOUT, SW17.DIN
- new net: SW17.DOUT, SW18.DIN
- new net: SW1.DOUT, SW2.DIN
- new net: SW8.DOUT, SW9.DIN
- new net: SW10.DIN, SW9.DOUT
- new net: SW23.DOUT, SW24.DIN
- new net: SW24.DOUT, SW25.DIN
- new net: SW11.DOUT, SW12.DIN
- new net: SW12.DOUT, SW13.DIN
- new net: SW2.DOUT, SW3.DIN
- new net: SW3.DOUT, SW4.DIN
- new net: SW22.DOUT, SW23.DIN
- new net: SW4.DOUT, SW5.DIN
- new net: SW18.DOUT, SW19.DIN
- new net: SW6.DOUT, SW7.DIN
- new net: SW7.DOUT, SW8.DIN
- new net INT: U1.48 (~{INT}), U2.9 (PA7_A8_D8_SCK)
- new net LEDROW1: SW5.DOUT, SW6.DIN
- new net LEDROW2: SW10.DOUT, SW11.DIN
- new net LEDROW3: SW15.DOUT, SW16.DIN
- new net LEDROW4: SW20.DOUT, SW21.DIN
- new net OE: U1.23 (~{OE}), U2.8 (PB09_A7_D7_RX)
- new net R1G: SW1.G, U1.53 (IO0_1)
- new net R1R: SW1.R, U1.52 (IO0_0)
- new net R1U: SW1.U, U1.54 (IO0_2)
- new net R2G: SW5.G, U1.1 (IO0_4)
- new net R2R: SW5.R, U1.56 (IO0_3)
- new net R2U: SW5.U, U1.2 (IO0_5)
- new net SWCLK: P2.1, U2.18 (PA30_SWCLK)
- new net SWDIO: P1.1, U2.17 (PA31_SWDIO)
- new net Switch1: SW1.2 (Sw2), U1.8 (IO1_2)
- new net Switch10: SW10.2 (Sw2), U1.40 (IO4_1)
- new net Switch11: SW11.2 (Sw2), U1.10 (IO1_4)
- new net Switch12: SW12.2 (Sw2), U1.17 (IO2_1)
- new net Switch13: SW13.2 (Sw2), U1.26 (IO2_6)
- new net Switch14: SW14.2 (Sw2), U1.33 (IO3_3)
- new net Switch15: SW15.2 (Sw2), U1.41 (IO4_2)
- new net Switch16: SW16.2 (Sw2), U1.12 (IO1_5)
- new net Switch17: SW17.2 (Sw2), U1.18 (IO2_2)
- new net Switch18: SW18.2 (Sw2), U1.28 (IO2_7)
- new net Switch19: SW19.2 (Sw2), U1.34 (IO3_4)
- new net Switch2: SW2.2 (Sw2), U1.14 (IO1_7)
- new net Switch20: SW20.2 (Sw2), U1.42 (IO4_3)
- new net Switch21: SW21.2 (Sw2), U1.13 (IO1_6)
- new net Switch22: SW22.2 (Sw2), U1.19 (IO2_3)
- new net Switch23: SW23.2 (Sw2), U1.29 (IO3_0)
- new net Switch24: SW24.2 (Sw2), U1.35 (IO3_5)
- new net Switch25: SW25.2 (Sw2), U1.43 (IO4_4)
- new net Switch3: SW3.2 (Sw2), U1.24 (IO2_4)
- new net Switch4: SW4.2 (Sw2), U1.30 (IO3_1)
- new net Switch5: SW5.2 (Sw2), U1.38 (IO4_0)
- new net Switch6: SW6.2 (Sw2), U1.9 (IO1_3)
- new net Switch7: SW7.2 (Sw2), U1.15 (IO2_0)
- new net Switch8: SW8.2 (Sw2), U1.25 (IO2_5)
- new net Switch9: SW9.2 (Sw2), U1.31 (IO3_2)
Other:
- moved on the sheet: C1, LED1, LED2, LED3, LED4, LED5, LED6, LED7, LED8

Commit message: seeed board changes
Connections:
- net Earth: now also U1.~
Changed lines of the file:
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@@
     (stroke (width 0) (type default) (color 0 0 0 0))
   )
+  (wire (pts (xy 327.152 83.82) (xy 322.58 83.82))
+    (stroke (width 0) (type default) (color 0 0 0 0))
+  )
   (wire (pts (xy 85.09 56.134) (xy 101.6 56.134))
     (stroke (width 0) (type default) (color 0 0 0 0))
@@
     (stroke (width 0) (type default) (color 0 0 0 0))
   )
+  (wire (pts (xy 395.986 108.204) (xy 388.62 108.204))
+    (stroke (width 0) (type default) (color 0 0 0 0))
+  )
   (wire (pts (xy 316.23 72.39) (xy 323.342 72.39))
     (stroke (width 0) (type default) (color 0 0 0 0))
   )
+  (wire (pts (xy 243.078 78.994) (xy 241.046 78.994))
+    (stroke (width 0) (type default) (color 0 0 0 0))
+  )
   (wire (pts (xy 341.63 185.166) (xy 246.38 185.166))
     (stroke (width 0) (type default) (color 0 0 0 0))
@@
     (stroke (width 0) (type default) (color 0 0 0 0))
   )
+  (wire (pts (xy 243.078 71.374) (xy 241.046 71.374))
+    (stroke (width 0) (type default) (color 0 0 0 0))
+  )
   (wire (pts (xy 246.38 199.39) (xy 254 199.39))
     (stroke (width 0) (type default) (color 0 0 0 0))
@@
     (stroke (width 0) (type default) (color 0 0 0 0))
   )
+  (wire (pts (xy 326.39 87.63) (xy 322.58 87.63))
+    (stroke (width 0) (type default) (color 0 0 0 0))
+  )
   (wire (pts (xy 252.73 56.896) (xy 246.38 56.896))
     (stroke (width 0) (type default) (color 0 0 0 0))
@@
     (pin "4")
   )
-  (symbol (lib_id "power:Earth") (at 241.046 78.994 90) (unit 1)
+  (symbol (lib_id "power:Earth") (at 243.078 78.994 90) (unit 1)
     (in_bom yes) (on_board yes)
-    (property "Reference" "#GND012" (id 0) (at 244.856 78.994 0)
+    (property "Reference" "#GND012" (id 0) (at 246.888 78.994 0)
       (effects (font (size 1.27 1.27)) hide)
     )
-    (property "Value" "Earth" (id 1) (at 244.856 78.994 0)
+    (property "Value" "Earth" (id 1) (at 246.888 78.994 0)
       (effects (font (size 1.27 1.27)) hide)
     )
-    (property "Footprint" "" (id 2) (at 241.046 78.994 0)
+    (property "Footprint" "" (id 2) (at 243.078 78.994 0)
       (effects (font (size 1.27 1.27)) hide)
     )
-    (property "Datasheet" "~" (id 3) (at 241.046 78.994 0)
+    (property "Datasheet" "~" (id 3) (at 243.078 78.994 0)
       (effects (font (size 1.27 1.27)) hide)
     )
@@
     (pin "1")
   )
-  (symbol (lib_id "eec:PCA9506BS,118") (at 363.22 104.648 0) (unit 2)
+  (symbol (lib_name "PCA9506BS,118_1") (lib_id "eec:PCA9506BS,118") (at 363.22 104.648 0) (unit 2)
     (in_bom yes) (on_board yes) (fields_autoplaced)
     (property "Reference" "U1" (id 0) (at 377.19 97.028 0))
@@
     (pin "55")
     (pin "57")
+    (pin "~")
   )
   (symbol (lib_id "SparkFun-PowerSymbols:5V") (at 63.5 203.2 90) (unit 1)
@@
     (pin "4")
   )
+  (symbol (lib_id "power:Earth") (at 395.986 108.204 90) (unit 1)
+    (in_bom yes) (on_board yes)
+    (property "Reference" "#GND0109" (id 0) (at 401.574 108.204 90)
+      (effects (font (size 1.27 1.27)) hide)
+    )
+    (property "Value" "Earth" (id 1) (at 399.796 108.204 0)
+      (effects (font (size 1.27 1.27)) hide)
+    )
+    (property "Footprint" "" (id 2) (at 395.986 108.204 0)
+      (effects (font (size 1.27 1.27)) hide)
+    )
+    (property "Datasheet" "~" (id 3) (at 395.986 108.204 0)
+      (effects (font (size 1.27 1.27)) hide)
+    )
+    (pin "1")
+  )
   (symbol (lib_id "power:Earth") (at 48.006 254 90) (unit 1)
     (in_bom yes) (on_board yes)
@@
     (pin "1")
   )
-  (symbol (lib_id "SparkFun-PowerSymbols:5V") (at 241.046 71.374 270) (unit 1)
+  (symbol (lib_id "SparkFun-PowerSymbols:5V") (at 243.078 71.374 270) (unit 1)
     (in_bom yes) (on_board yes)
-    (property "Reference" "#SUPPLY0102" (id 0) (at 241.046 72.644 0)
+    (property "Reference" "#SUPPLY0102" (id 0) (at 243.078 72.644 0)
       (effects (font (size 1.143 1.143)) (justify left bottom) hide)
     )
-    (property "Value" "5V" (id 1) (at 244.094 70.104 0)
+    (property "Value" "5V" (id 1) (at 246.126 70.104 0)
       (effects (font (size 1.143 1.143)) (justify left bottom))
     )
-    (property "Footprint" "XXX-00000" (id 2) (at 248.666 71.374 0)
+    (property "Footprint" "XXX-00000" (id 2) (at 250.698 71.374 0)
       (effects (font (size 1.524 1.524)) hide)
     )
-    (property "Datasheet" "" (id 3) (at 241.046 71.374 0)
+    (property "Datasheet" "" (id 3) (at 243.078 71.374 0)
       (effects (font (size 1.524 1.524)) hide)
     )
@@
     (pin "~")
   )
-  (symbol (lib_id "power:Earth") (at 322.58 87.63 90) (unit 1)
+  (symbol (lib_id "power:Earth") (at 326.39 87.63 90) (unit 1)
     (in_bom yes) (on_board yes)
-    (property "Reference" "#GND014" (id 0) (at 328.168 87.63 90))
-    (property "Value" "Earth" (id 1) (at 326.39 87.63 0)
+    (property "Reference" "#GND014" (id 0) (at 335.534 87.63 90))
+    (property "Value" "Earth" (id 1) (at 330.2 87.63 0)
       (effects (font (size 1.27 1.27)) hide)
     )
-    (property "Footprint" "" (id 2) (at 322.58 87.63 0)
+    (property "Footprint" "" (id 2) (at 326.39 87.63 0)
       (effects (font (size 1.27 1.27)) hide)
     )
-    (property "Datasheet" "~" (id 3) (at 322.58 87.63 0)
+    (property "Datasheet" "~" (id 3) (at 326.39 87.63 0)
       (effects (font (size 1.27 1.27)) hide)
     )
@@
     (pin "~")
   )
-  (symbol (lib_id "SparkFun-PowerSymbols:5V") (at 322.58 83.82 270) (unit 1)
+  (symbol (lib_id "SparkFun-PowerSymbols:5V") (at 327.152 83.82 270) (unit 1)
     (in_bom yes) (on_board yes)
-    (property "Reference" "#SUPPLY011" (id 0) (at 322.58 85.09 0)
+    (property "Reference" "#SUPPLY011" (id 0) (at 327.152 85.09 0)
       (effects (font (size 1.143 1.143)) (justify left bottom) hide)
     )
-    (property "Value" "5V" (id 1) (at 326.39 84.836 90)
+    (property "Value" "5V" (id 1) (at 330.962 84.836 90)
       (effects (font (size 1.143 1.143)) (justify left bottom))
     )
-    (property "Footprint" "XXX-00000" (id 2) (at 330.2 83.82 0)
+    (property "Footprint" "XXX-00000" (id 2) (at 334.772 83.82 0)
       (effects (font (size 1.524 1.524)) hide)
     )
-    (property "Datasheet" "" (id 3) (at 322.58 83.82 0)
+    (property "Datasheet" "" (id 3) (at 327.152 83.82 0)
       (effects (font (size 1.524 1.524)) hide)
     )
@@
       (reference "#GND0108") (unit 1) (value "Earth") (footprint "")
     )
+    (path "/71ae337c-84a1-433b-ad69-ceecbb1d2b0c"
+      (reference "#GND0109") (unit 1) (value "Earth") (footprint "")
+    )
     (path "/26b3b00b-2013-4fc7-b50e-a5e0ba544b49"
